Commit message: updated ceres urdf file

File: robot_description/urdf/ceres.urdf (robot description, URDF)
Before this commit: robot ceres_rover, 3 links, 2 joints
Links:
- removed link arm_base_link
- removed link shoulder_assembly_link
- added link base_pivot_link; visual mesh filename=package://robot_description/meshes/arm_parts/cycloidal_driv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 scale=0.001 0.001 0.001
- added link base_structure_link; visual mesh filename=package://robot_description/meshes/arm_parts/cycloidal_driv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 scale=0.001 0.001 0.001
- added link bicep_gearbox_link; visual mesh filename=package://robot_description/meshes/arm_parts/cycloidal_driv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 scale=0.001 0.001 0.001
- added link forearm_tube_link; visual mesh filename=package://robot_description/meshes/arm_parts/cycloidal_driv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 scale=0.001 0.001 0.001
- added link shoulder_gearbox_link; visual mesh filename=package://robot_description/meshes/arm_parts/cycloidal_driv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 scale=0.001 0.001 0.001
- link bicep_tube_link: geometry visual mesh filename=package://robot_description/meshes/arm_parts/cycloidal_driv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 scale=0.001 0.001 0.001
Joints:
- removed joint arm_shoulder_joint
- removed joint bicep_tube_shoulder_assembly_joint
- added joint base_pivot_shoulder_gearbox_joint: type continuous, parent base_pivot_link, child shoulder_gearbox_link, origin xyz=0 0 0.082 rpy=0 0 0, axis 1 0 0
- added joint base_structure_joint: type continuous, parent base_structure_link, child base_pivot_link, origin xyz=0.156 -0.074 0.104 rpy=0 0 0, axis 0 0 1
- added joint bicep_gearbox_forearm_tube_joint: type fixed, parent bicep_gearbox_link, child forearm_tube_link, origin xyz=0 0 0 rpy=0 0 0
- added joint bicep_tube_gearbox_joint: type continuous, parent bicep_tube_link, child bicep_gearbox_link, origin xyz=0.0837 -0.238 0.3750 rpy=0 0 0, axis 1 0 0
- added joint shoulder_tube_joint: type fixed, parent shoulder_gearbox_link, child bicep_tube_link, origin xyz=0 0 0 rpy=0 0 0

Commit message: almost complete version of arm

File: robot_description/urdf/ceres.urdf (robot description, URDF)
Before this commit: robot ceres_rover, 6 links, 5 joints
Links:
- added link forearm_gearbox_link; visual mesh filename=package://robot_description/meshes/arm_parts/cycloidal_driv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 scale=0.001 0.001 0.001
- added link gripper_claw_link; visual mesh filename=package://robot_description/meshes/arm_parts/cycloidal_driv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 scale=0.001 0.001 0.001
- added link gripper_gearbox_link; visual mesh filename=package://robot_description/meshes/arm_parts/cycloidal_driv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 scale=0.001 0.001 0.001
- added link wrist_gearbox_link; visual mesh filename=package://robot_description/meshes/arm_parts/cycloidal_driv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 scale=0.001 0.001 0.001
Joints:
- added joint forearm_gearbox_joint: type fixed, parent forearm_tube_link, child forearm_gearbox_link, origin xyz=0 0 0 rpy=0 0 0
- added joint forearm_tube_wrist_gearbox_joint: type continuous, parent forearm_tube_link, child wrist_gearbox_link, origin xyz=0 0 0.345 rpy=0 0 0, axis  1 0 0
- added joint gripper_claw_joint: type continuous, parent gripper_gearbox_link, child gripper_claw_link, origin xyz=0 -0.11 0 rpy=0 0 0, axis 0 1 0
- added joint wrist_gearbox_gripper_gearbox_joint: type fixed, parent wrist_gearbox_link, child gripper_gearbox_link, origin xyz=0 0 0 rpy=0 0 0
- joint bicep_gearbox_forearm_tube_joint: axis (none) ->  0 0 1; origin xyz=0 0 0 rpy=0 0 0 -> xyz=-0.09562 -0.058 0.01 rpy=2.181 0 0; type fixed -> continuous
- joint bicep_tube_gearbox_joint: origin xyz=0.0837 -0.238 0.3750 rpy=0 0 0 -> xyz=0.0837 -0.224 0.3530 rpy=0 0 0
